File: mesh/mesh.kicad_sch (KiCad schematic)
At the start: 77 parts, among them J1 SMA edge, J2 USB-A edge fingers, SW1 USER, SW2 BOOTSEL, U1 RP2040, U2 SX1262IMLTRT, U3 GD25Q32E, U4 PE4259-63, U5 ME6211C33M5G, U6 LP5907MFX-3.3, U7 USBLC6-2SC6, U8 74HCT2G34, Y1 12MHz, Y2 32MHz TCXO clipped-sine

Commit message: Rev B: USB-C plug, red-team fixes, and a schematic that reads as one
USB-A edge fingers are gone; J2 is a real USB-C male plug. A sink presenting a
plug terminates CC with a SINGLE Rd -- putting 5.1k on both CC and VCONN shows the
host the Debug Accessory signature instead of a device. All four VBUS and all four
GND contacts bus through. B6/B7, SBU and the SuperSpeed pads are deliberately
unnetted, per Type-C R2.4 Table 3-11 notes 2 and 5.

The plug is a straddle mount -- the A row lands on F.Cu, the B row on B.Cu, and the
board edge becomes the plug's tongue -- so the CONNECTOR now sets the stack-up at
0.8 mm. That is also what makes a 90 ohm USB pair and a sane 50 ohm RF line
routable on a 20 mm-wide board, which 2.0 mm never was.

Defects found by review and fixed, each against a primary source:

  - No 1 uF at VREG_VIN. The RP2040 core LDO needs one at BOTH ends.
  - One 100 nF across two DVDD pins on opposite corners of the QFN, and nothing
    at all on USB_VDD or ADC_AVDD. The six caps exactly consumed the six IOVDD
    pins.
  - No pull-up on QSPI_SS. CS# must be at its own supply through the 3V3 ramp, and
    RPi only omit it for a flash they qualified -- which the GD25Q32E is not.
  - 27 pF crystal loads tagged [rpi], but Raspberry Pi's value is 15 pF for a
    CL=10 pF part. 27 pF implies CL=16.5 pF, which matches no specified crystal and
    eats start-up margin. Y1 now names one.
  - 55 uF on VBUS against a 10 uF ceiling in BOTH USB 2.0 and Type-C. Values only,
    no footprint changes: now 9.1 uF.
  - Y2 was an HCMOS oscillator symbol with pin 1 driven as an enable. A clipped-sine
    TCXO has NC there. The 2520 body is also where the cheap 32 MHz parts live.
  - C40/R6 swapped to Semtech Fig 4-2 order, and the ESD array got the bypass its
    datasheet asks for at pin 5.

BOM reductions, all of which also remove risk:

  - SK9822 + 74HCT2G34 + support -> two plain LEDs. Upstream Meshtastic has no
    APA102/SK9822 driver at all, so the old chain neede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
Parts:
- removed AE1: IFA 915MHz, zach:Antenna_IFA_915MHz, symbol Connector_Generic:Conn_01x01
- removed C38: 100n, Capacitor_SMD:C_0402_1005Metric, symbol Device:C
- removed C39: 10u, Capacitor_SMD:C_0603_1608Metric, symbol Device:C
- removed RA, RB: 0R, Resistor_SMD:R_0402_1005Metric, symbol Device:R
- removed SW2: BOOTSEL, Button_Switch_SMD:SW_Push_1P1T_XKB_TS-1187A, symbol Switch:SW_Push
- removed U8: 74HCT2G34, Package_TO_SOT_SMD:SOT-363_SC-70-6, symbol 74xGxx:74AUC2G34
- added C41, C43, C44: 100n, Capacitor_SMD:C_0402_1005Metric, symbol Device:C
- added C42: 1u, Capacitor_SMD:C_0402_1005Metric, symbol Device:C
- added D2: red, LED_SMD:LED_0603_1608Metric, symbol Device:LED
- added R11: 5k1, Resistor_SMD:R_0402_1005Metric, symbol Device:R
- added R14: 10k, Resistor_SMD:R_0402_1005Metric, symbol Device:R
- added TP4: RUN, TestPoint:TestPoint_Pad_D1.0mm, symbol Connector:TestPoint
- added TP5: BOOTSEL, TestPoint:TestPoint_Pad_D1.0mm, symbol Connector:TestPoint
- added TP6: SDA, TestPoint:TestPoint_Pad_D1.0mm, symbol Connector:TestPoint
- added TP7: SCL, TestPoint:TestPoint_Pad_D1.0mm, symbol Connector:TestPoint
- C1, C2: value 27p -> 15p
- C11: value 100n -> 1u
- C26: value 22u -> 4u7; footprint Capacitor_SMD:C_0805_2012Metric -> Capacitor_SMD:C_0603_1608Metric
- C27: value 22u -> 1u; footprint Capacitor_SMD:C_0805_2012Metric -> Capacitor_SMD:C_0402_1005Metric
- D1: value SK9822-EC20 -> green; footprint zach:LED_SK9822-EC20_2020 -> LED_SMD:LED_0603_1608Metric; symbol zach:SK9822-EC20 -> Device:LED; MPN SK9822-EC20 -> (none)
- J2: value USB-A edge fingers -> USB-C plug; footprint zach:USB_A_EdgeFinger_2.0mm -> Connector_USB:USB_C_Plug_JAE_DX07P024AJ1; symbol Connector:USB_A -> Connector:USB_C_Plug_USB2.0
- R10, R9: value 100R -> 1k
- U1: footprint Package_DFN_QFN:QFN-56-1EP_7x7mm_P0.4mm_EP3.2x3.2mm -> zach:RP2040-QFN-56-1EP_7x7mm_P0.4mm_EP-vias
- U2: footprint Package_DFN_QFN:QFN-24-1EP_4x4mm_P0.5mm_EP2.6x2.6mm -> zach:SX1262-QFN-24-1EP_4x4mm_P0.5mm_EP-vias
- Y1: value 12MHz -> 12MHz CL10p; MPN (none) -> ABM8-272-T3; Manufacturer (none) -> Abracon
- Y2: value 32MHz TCXO clipped-sine -> 32MHz TCXO 1.8V clipped-sine; footprint Oscillator:Oscillator_SMD_Abracon_ASE-4Pin_3.2x2.5mm -> Oscillator:Oscillator_SMD_SeikoEpson_TG2520SMN-xxx-xxxxxx-4Pin_2.5x2.0mm; symbol Oscillator:ASE-xxxMHz -> Oscillator:TG2520SMN-xx.xxxxxxMhz-xxxxNM; LCSC (none) -> C7527388; MPN (none) -> TG2520SMN 32.0000M; Manufacturer (none) -> Seiko Epson
Connections:
- net ANT_SMA is gone; now on net ANT2: J1.1 (In)
- net LED_CLK_5V is gone; now on net LED_PWR_K: R9.1
- net +3V3: now also C42.1, C44.1, R14.1
- net BOOT_SW: now also TP5.1
- net DVDD: now also C43.1
- net GND: now also J2.A1 (GND), J2.A12 (GND), J2.B1 (GND), J2.B12 (GND), R10.2, R9.2, C41.2, C42.2, C43.2, C44.2, R11.2; no longer D1.2 (GND), J2.4 (GND)
- net QSPI_SS: now also R14.2
- net RUN: now also TP4.1
- net TCXO_AC: now also C40.1, R6.2; no longer C40.2, R6.1
- net TCXO_OUT: now also R6.1; no longer C40.1
- net USB_DM_C: now also J2.A7 (D-); no longer J2.2 (D-)
- net USB_DM_R: no longer R1.2, U1.47 (USB_DP)
- net USB_DP_C: now also J2.A6 (D+); no longer J2.3 (D+)
- net VBUS: now also J2.A4 (VBUS), J2.A9 (VBUS), J2.B4 (VBUS), J2.B9 (VBUS), C41.1; no longer D1.5 (VDD), J2.1 (VBUS)
- net VDD_TCXO: no longer Y2.1 (EN)
- net XTA: now also C40.2; no longer R6.2
- net I2C_SDA: now reaches U1.6 (GPIO4)
- net I2C_SDA: now also TP6.1
- net I2C_SCL: now reaches U1.7 (GPIO5)
- net I2C_SCL: now also TP7.1
- net LED_PWR_K: now reaches D1.1 (K)
- removed net CKI: D1.4 (CKI), R9.2
- net LED_CLK renamed LED_PWR
- net LED_PWR: now also D1.2 (A)
- net LED_DAT renamed LED_LORA
- net LED_LORA: now also D2.2 (A)
- net LED_DAT_5V renamed LED_LORA_K
- net LED_LORA_K: now also D2.1 (K)
- removed net SDI: D1.3 (SDI), R10.2
- new net USB_CC: J2.A5 (CC), R11.1
- new net USB_DP: R1.2, U1.47 (USB_DP)
- no-connect marks 25 -> 23
Other:
- note added: "A USB-C plug entry, ESD, power rails"
- note added: "B RP2040, QSPI flash, crystal, buttons"
- note added: "E Status LEDs: heartbeat and radio activity"
- note removed: "A USB entry, ESD, power rails"
- note removed: "B RP2040, flash, crystal, buttons"
- note removed: "E SK9822 activity LED, 5V logic via HCT buffer"
- title: Pikkolo Mesh Stick Rev A -> Pikkolo Mesh Stick
- moved on the sheet: C1, C10, C11, C12, C13, C14, C15, C16, C17, C18, C19, C2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

Commit message: Adopt the Johanson IPD, go 4-layer, and fix two bugs Rev B introduced
A fresh-eyes review found that the Rev B bulk-cap cut had created a defect. With the
VBUS bulk trimmed to spec, FB1 was left driving only 2 uF: a 0.6-1.6 uH bead against
2 uF is a 90-145 kHz tank damped only by its own DCR, and a hot-plug step rings 13-49%
above 5 V -- past the LP5907's 6.0 V absolute maximum. The ferrite is deleted and both
LDO inputs now sit on the node the ESD array actually clamps. That also closes
DECISIONS['ferrite_fb1'].

Second bug from the same change set: the I2C pads added for expansion had no pull-ups
anywhere. I2C is open drain, so the bus could never be released high, and the RP2040's
50-80k internal pull-up gives a 15-25 us rise into even 100 pF. R12/R13 4k7 added.

RF FRONT END. The discrete matching network is replaced by one part, FL1. What was
there was Semtech's SX1261 topology being run at +22 dBm -- two elements short of their
SX1262 network -- with values copied from a licensee's schematic and never validated,
on a 20 mm-wide stick that would have needed a VNA campaign to tune. The IPD's response
is fixed in LTCC and factory-tested, and it replaces the TX filter AND the RX balun.

The K variant, not the D, and the reason is regulatory: 2f0 is NOT in an FCC restricted
band and needs only 20 dBc, but 3f0, 4f0 and 5f0 all are and need ~63 dB. The D part
specifies nothing above 3f0. The K specifies all three, and swallows the antenna pi as
well -- whose lands stay as a stuffing option with R15 linking them out.

No library work was needed: KiCad 10 already ships Filter:0900FM15K0039 and
RF_Converter:Balun_Johanson_0900FM15K0039. The part is DigiKey-only, so it is consigned
or hand-placed if this goes to JLCPCB assembly.

STACK-UP resolved to 4 layers, JLC04081H-3313, which is a fee-free JLCPCB option. The
buy is not lower via inductance -- a reviewer recomputed that argument and it does not
survive contact with 0.8 mm, where the resonances land at 2.2-3.9 GHz an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
Parts:
- removed C20: 3p, Capacitor_SMD:C_0402_1005Metric, symbol Device:C
- removed C21: 5p6, Capacitor_SMD:C_0402_1005Metric, symbol Device:C
- removed C23, C31: 1p8, Capacitor_SMD:C_0402_1005Metric, symbol Device:C
- removed C24: 1p, Capacitor_SMD:C_0402_1005Metric, symbol Device:C
- removed FB1: 600R@100MHz, Inductor_SMD:L_0603_1608Metric, symbol Device:FerriteBead
- removed L2: 2n5, Inductor_SMD:L_0402_1005Metric, symbol Device:L
- removed L3: 4n7, Inductor_SMD:L_0402_1005Metric, symbol Device:L
- removed L4: 15n, Inductor_SMD:L_0402_1005Metric, symbol Device:L
- removed L5: 9n1, Inductor_SMD:L_0402_1005Metric, symbol Device:L
- added FL1: 0900FM15K0039001E, RF_Converter:Balun_Johanson_0900FM15K0039, symbol Filter:0900FM15K0039
- added R12, R13: 4k7, Resistor_SMD:R_0402_1005Metric, symbol Device:R
- added R15: 0R, Resistor_SMD:R_0402_1005Metric, symbol Device:R
- C25: value 2p4 -> 39p
- C33, C34: now not fitted
- R10, R9: value 1k -> 470R
- Y2: MPN TG2520SMN 32.0000M -> TG2520SMN 32.0000M-ECGNNM
Connections:
- net TX2 is gone; now on net RF_TX: C22.2
- net VBUS_F is gone; now on net VBUS: C15.1, C27.1, U5.1 (V_{IN}), U5.3 (CE), U6.1 (IN), U6.3 (EN)
- net +3V3: now also R12.1, R13.1
- net ANT1: now also R15.1
- net ANT2: now also R15.2
- net GND: now also FL1.10 (GND), FL1.2 (GND), FL1.5 (GND), FL1.7 (GND), FL1.9 (GND)
- net I2C_SCL: now also R13.2
- net I2C_SDA: now also R12.2
- net RFI_N: now also FL1.3 (RFI_N); no longer C25.2
- net RFI_P: now also FL1.4 (RFI_P)
- net RFO: now also FL1.1 (RFO)
- net RF_RX: now also C25.2; no longer C25.1
- net TX1 renamed IPD_TX
- net IPD_TX: now also FL1.8 (SW_RFO)
- new net IPD_RX: C25.1, FL1.6 (SW_RFI)
Other:
- note added: "D Johanson IPD front end + SPDT antenna switch 902-928MHz"
- note removed: "D TX LPF / RX balun / antenna pi / SPDT values [ws] 902-928MHz - tune on hardware"
- moved on the sheet: C22, C25, C32, C35, C36, J1, R7, R8

Commit message: Close the flash and antenna decisions, and source the BOM
FLASH, respin class. The GD25Q32E accepts only a one-byte 01h Write Status Register.
The RP2040's stock second stage issues 01h followed by TWO data bytes in one CS#
assertion, which that datasheet says is not executed at all -- so the quad-enable bit
stays 0, the EBh quad read returns garbage, and the chip faults out of boot2. The
symptom is the nastiest kind available: the board enumerates as RPI-RP2 and happily
accepts a UF2, then never runs.

U3 becomes W25Q128JVSIQ. The Winbond "...IQ" order codes ship with QE already fixed to
1 in silicon, so boot2's 35h check short-circuits and the offending write is never
issued -- the bug class cannot occur rather than being worked around. It is also a
JLCPCB Basic part, so no extended-part fee and no stock roulette. Pin-for-pin identical
to the symbol it replaces; the stock 208-mil SOIC-8 footprint is unchanged. That also
retires the planned dual 150/208-mil custom footprint, which would have put 2.9 mm pads
on six nets clocking at sysclk/2 to buy an option nobody needs.

ANTENNA. Not a board-edge SMA. Two edge connectors would have to share one thickness
window and they do not: the JAE plug needs 0.72-0.88 mm, the only orderable 0.8 mm
end-launch SMA caps at 0.79 mm, and the fab delivers 0.72-0.88 mm -- a tolerance wider
than the parts allow, on a $3.40 hand-solder part that cantilevers a brass cube on a
13 mm lever off the edge of a 0.8 mm board living in a laptop port. J1 is a u.FL
receptacle: surface mount, thickness-agnostic, $0.23, machine-placeable, and the strain
path moves to the enclosure where it belongs. The bulkhead must be a standard SMA
FEMALE jack -- Meshtastic whips are SMA male, not RP-SMA.

TCXO. Switched to the 3.0 V ordering code (MCGNNM). The 1.8 V sibling is specified
1.7-1.9 V and RadioLib's SX126x default tcxoVoltage is 1.6 V, below its minimum -- one
firmware slip and the radio never starts. At 3.0 V, VBAT 3.3 V still satisfies
VBAT >= VTCX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
Parts:
- C1, C2: Dielectric (none) -> C0G; LCSC (none) -> C1548; MPN (none) -> 0402CG150J500NT; Manufacturer (none) -> FH; Tolerance (none) -> 5%; Voltage (none) -> 50V
- C10, C12, C13, C14, C3, C4, C41, C43, C44, C5, C6, C7, C8, C9: Dielectric (none) -> X7R; LCSC (none) -> C1525; MPN (none) -> CL05B104KO5NNNC; Manufacturer (none) -> Samsung; Tolerance (none) -> 10%; Voltage (none) -> 16V
- C11, C15, C16, C17, C27, C28, C42: Dielectric (none) -> X5R; LCSC (none) -> C52923; MPN (none) -> CL05A105KA5NQNC; Manufacturer (none) -> Samsung; Tolerance (none) -> 10%; Voltage (none) -> 25V
- C18, C19: value 10u -> 4u7; Dielectric (none) -> X5R; LCSC (none) -> C19666; MPN (none) -> CL10A475KO8NNNC; Manufacturer (none) -> Samsung; Tolerance (none) -> 10%; Voltage (none) -> 16V
- C22, C25, C32: Dielectric (none) -> NP0; LCSC (none) -> C106223; MPN (none) -> CC0402JRNPO9BN390; Manufacturer (none) -> YAGEO; Tolerance (none) -> 5%; Voltage (none) -> 50V
- C26: Dielectric (none) -> X5R; LCSC (none) -> C19666; MPN (none) -> CL10A475KO8NNNC; Manufacturer (none) -> Samsung; Tolerance (none) -> 10%; Voltage (none) -> 16V
- C29: Dielectric (none) -> X5R; LCSC (none) -> C47339; MPN (none) -> CL05A474KP5NNNC; Manufacturer (none) -> Samsung; Tolerance (none) -> 10%; Voltage (none) -> 10V
- C30: Dielectric (none) -> X7R; LCSC (none) -> C285062; MPN (none) -> 0402B473K250NT; Manufacturer (none) -> FH; Tolerance (none) -> 10%; Voltage (none) -> 25V
- C33, C34: Dielectric (none) -> C0G; LCSC (none) -> C76907; MPN (none) -> GJM1555C1H3R9BB01D; Manufacturer (none) -> Murata; Tolerance (none) -> +/-0.1pF; Voltage (none) -> 50V
- C35, C36: Dielectric (none) -> X7R; LCSC (none) -> C1523; MPN (none) -> 0402B102K500NT; Manufacturer (none) -> FH; Tolerance (none) -> 10%; Voltage (none) -> 50V
- C37: value 47p -> 39p; Dielectric (none) -> NP0; LCSC (none) -> C106223; MPN (none) -> CC0402JRNPO9BN390; Manufacturer (none) -> YAGEO; Tolerance (none) -> 5%; Voltage (none) -> 50V
- C40: Dielectric (none) -> C0G; LCSC (none) -> C32949; MPN (none) -> CL05C100JB5NNNC; Manufacturer (none) -> Samsung; Tolerance (none) -> 5%; Voltage (none) -> 50V
- D1: LCSC (none) -> C965805; MPN (none) -> XL-1608SYGC-06; Manufacturer (none) -> XINGLIGHT
- D2: LCSC (none) -> C2286; MPN (none) -> KT-0603R; Manufacturer (none) -> Hubei KENTO
- J1: value SMA edge -> u.FL; footprint Connector_Coaxial:SMA_Amphenol_132289_EdgeMount -> Connector_Coaxial:U.FL_Hirose_U.FL-R-SMT-1_Vertical; LCSC (none) -> C88373; MPN (none) -> U.FL-R-SMT-1(10); Manufacturer (none) -> Hirose
- J2: LCSC (none) -> C5352764; MPN (none) -> DX07P024AJ1R1500; Manufacturer (none) -> JAE
- L1: LCSC (none) -> C237556; MPN (none) -> LQW15AN47NG80D; Manufacturer (none) -> Murata; Tolerance (none) -> 2%
- R1, R2: LCSC (none) -> C25100; MPN (none) -> 0402WGF270JTCE; Manufacturer (none) -> UNI-ROYAL; Tolerance (none) -> 1%
- R11: LCSC (none) -> C25905; MPN (none) -> 0402WGF5101TCE; Manufacturer (none) -> UNI-ROYAL; Tolerance (none) -> 1%
- R14, R5: LCSC (none) -> C25744; MPN (none) -> 0402WGF1002TCE; Manufacturer (none) -> UNI-ROYAL; Tolerance (none) -> 1%
- R3, R4: LCSC (none) -> C11702; MPN (none) -> 0402WGF1001TCE; Manufacturer (none) -> UNI-ROYAL; Tolerance (none) -> 1%
- R6: LCSC (none) -> C25091; MPN (none) -> 0402WGF2200TCE; Manufacturer (none) -> UNI-ROYAL; Tolerance (none) -> 1%
- R7, R8: LCSC (none) -> C25076; MPN (none) -> 0402WGF1000TCE; Manufacturer (none) -> UNI-ROYAL; Tolerance (none) -> 1%
- SW1: LCSC (none) -> C318884; MPN (none) -> TS-1187A-B-A-B; Manufacturer (none) -> XKB
- TP1, TP2, TP3, TP4, TP5, TP6, TP7: now left out of the parts list
- U1: LCSC (none) -> C2040; MPN (none) -> RP2040; Manufacturer (none) -> Raspberry Pi
- U2: LCSC (none) -> C191341; MPN (none) -> SX1262IMLTRT; Manufacturer (none) -> Semtech
- U3: value GD25Q32E -> W25Q128JVSIQ; symbol zach:GD25Q32E -> Memory_Flash:W25Q128JVS; LCSC (none) -> C97521; MPN (none) -> W25Q128JVSIQ; Manufacturer (none) -> Winbond
- U4: LCSC (none) -> C470892
- U5: LCSC (none) -> C82942; MPN (none) -> ME6211C33M5G-N; Manufacturer (none) -> Microne
- U6: LCSC (none) -> C80670; MPN (none) -> LP5907MFX-3.3/NOPB; Manufacturer (none) -> Texas Instruments
- U7: LCSC (none) -> C2687116; MPN (none) -> USBLC6-2SC6; Manufacturer (none) -> UMW
- Y1: LCSC (none) -> C20625731
- Y2: value 32MHz TCXO 1.8V clipped-sine -> 32MHz TCXO 3.0V clipped-sine; LCSC C7527388 -> C3007516; MPN TG2520SMN 32.0000M-ECGNNM -> TG2520SMN 32.000000M-MCGNNM

Commit message: Fix the QFN paste apertures, respecify the LDO capacitors, and record the fab constraints
The forked exposed-pad footprints had two manufacturability defects. Paste coverage was
47.3% (RP2040) and 39.8% (SX1262), both under IPC-7093A's 50-60% band for a thermal
land, and the apertures cleared the via barrels by 0.00 mm -- so paste would have wicked
straight down the holes. Vias are now 0.50/0.30 mm, which is also exactly the project's
0.10 mm minimum annular ring, and the apertures are retuned to 56.3% and 52.3% with
0.05 mm and 0.03 mm of barrel clearance. They stay ordinary plated through holes: the
fab's plugged-via rules exclude a via with a mask opening on either side, and the
exposed pad's own opening is one, so promising filled vias would be promising something
that cannot be delivered.

POWER. TI specify CIN >= 0.7 uF for the LP5907 "over the full range of operating
conditions", and a 1 uF 0402 sitting at 5-5.5 V of DC bias derates to 0.3-0.5 uF -- under
the floor, which is the kind of thing that shows up as an oscillating regulator nobody
can reproduce. C15 and C27 become 16 V 0603 4u7, one at each LDO input rather than a
shared bulk cap at the connector, which also satisfies TI's "not more than 1 cm from the
input pin". The separate bulk C26 goes away; total VBUS capacitance is 9.5 uF, still
inside the 10 uF spec ceiling. C14 is deleted as a duplicate of C10, which brings the
LP5907's output capacitance back under its 10 uF stability maximum.

The one-LDO-or-two question is now answered with a number rather than an adjective:
merged onto a single ME6211 the worst-case corner dissipates 432 mW against that
package's 300 mW ABSOLUTE MAXIMUM. Two LDOs is not a preference.

Recorded in the notes, because they are decisions that must survive into layout: order
the stack-up by name (the fab's thickness tolerance is wider than the connector's window
and only the nominal is controllable); specify a 0.12 mm stencil (the QFN-56's lead
apertures fall below IPC's 0.66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
Parts:
- removed C14: 100n, Capacitor_SMD:C_0402_1005Metric, symbol Device:C
- removed C26: 4u7, Capacitor_SMD:C_0603_1608Metric, symbol Device:C
- C15, C27: value 1u -> 4u7; footprint Capacitor_SMD:C_0402_1005Metric -> Capacitor_SMD:C_0603_1608Metric; LCSC C52923 -> C19666; MPN CL05A105KA5NQNC -> CL10A475KO8NNNC; Voltage 25V -> 16V
Other:
- moved on the sheet: C27

Commit message: Flash: W25Q32JVSSIQ, not W25Q128JVSIQ — and the sourcing objection checked
Pushed back on the Winbond choice on the grounds that Winbond flash is impossible to
find or discontinued, so I checked LCSC rather than argue:

  W25Q32JVSSIQ   C179173   70,003 in stock   $0.554   SOIC-8-208mil
  W25Q128JVSIQ   C97521    ~95,000           $2.45    SOIC-8-208mil, JLCPCB Basic
  GD25Q32ESIGR             37,921            $0.906

The scarcity does not hold for the JV generation. W25Q32JVSSIQ has nearly twice the
stock of the GigaDevice part it replaces and costs 40% less, at the same 4 MB and the
same 208-mil SOIC-8, with a pin-identical KiCad symbol.

Where the objection does hold: the other RP2040 board in this workspace fits
W25Q80DVUXIE, and that IS a genuinely awkward part — an older DV generation in USON-8,
superseded by JV/DW. Different part, different situation, and it is worth writing down
so this does not get re-litigated from memory next time.

So U3 becomes W25Q32JVSSIQ rather than the 16 MB part I picked last commit. It keeps the
whole reason for leaving GigaDevice -- the IQ order code fixes QE=1 in silicon, so the
stock RP2040 boot2 finds the bit already set and never issues the two-byte status-register
write that the GD25Q32E will not execute -- while being cheaper than either alternative
and matching the capacity that was actually specified. It is an Extended part rather than
Basic, which costs one ~$3 setup fee per order and is still far ahead on any run:
$8.54 against $24.50 for ten boards.

Co-Authored-By: Claude Opus 5 (1M context) <noreply@anthropic.com>
Claude-Session: https://claude.ai/code/session_01L6RoqgW9x4s4XgQCvcFbCH
Parts:
- U3: value W25Q128JVSIQ -> W25Q32JVSSIQ; symbol Memory_Flash:W25Q128JVS -> Memory_Flash:W25Q32JVSS; LCSC C97521 -> C179173; MPN W25Q128JVSIQ -> W25Q32JVSSIQ
Changed lines of the file:
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@@
 	)
 	(symbol
-		(lib_id "Memory_Flash:W25Q128JVS")
+		(lib_id "Memory_Flash:W25Q32JVSS")
 		(at 355.6 187.96 0)
 		(unit 1)
@@
 			)
 		)
-		(property "Value" "W25Q128JVSIQ"
+		(property "Value" "W25Q32JVSSIQ"
 			(at 345.44 165.1 0)
 			(show_name no)
@@
 			)
 		)
-		(property "Datasheet" "https://www.winbond.com/resource-files/w25q128jv_dtr%20revc%2003272018%20plus.pdf"
+		(property "Datasheet" "http://www.winbond.com/resource-files/w25q32jv%20revg%2003272018%20plus.pdf"
 			(at 355.6 187.96 0)
 			(hide yes)
@@
 			)
 		)
-		(property "Description" "16MB QSPI NOR flash, SOIC-8 208mil. QE fixed at 1 in silicon (IQ order code) so the stock RP2040 boot2 never issues its two-byte WRSR. JLCPCB Basic."
+		(property "Description" "4MB QSPI NOR flash, SOIC-8 208mil. The IQ order code fixes QE=1 in silicon, so the stock RP2040 boot2 finds the bit already set and never issues its two-byte WRSR. 70k at LCSC and cheaper than the GigaDevice part. NOT W25Q80DV -- that is the older generation, USON-8, and is the part that is genuinely hard to source."
 			(at 355.6 187.96 0)
 			(hide yes)
@@
 			)
 		)
-		(property "ki_keywords" "flash memory SPI QPI DTR"
+		(property "ki_keywords" "flash memory SPI"
 			(at 355.6 187.96 0)
 			(hide yes)
@@
 			)
 		)
-		(property "MPN" "W25Q128JVSIQ"
+		(property "MPN" "W25Q32JVSSIQ"
 			(at 355.6 187.96 0)
 			(hide yes)
@@
 			)
 		)
-		(property "LCSC" "C97521"
+		(property "LCSC" "C179173"
 			(at 355.6 187.96 0)
 			(hide yes)
